Commit message: new environment added

File: src/ur5_description/urdf/ur5.urdf.xacro (robot description, xacro)
@@ -99,5 +99,27 @@
       </collision>
   </link> -->
-    <link name="table">
+    <link name="pick_table">
+      <inertial>
+        <mass value="0.1" />
+        <inertia ixx="0.00" iyy="0.00" izz="0.00" ixy="0.0" ixz="0.0" iyz="0.0" />
+      </inertial>
+      <visual name="">
+        <origin xyz="0.0 0.0 0.0" rpy="0.0 0.0 0.0"/>
+        <geometry>
+          <mesh filename="package://ur5_description/meshes/ur5/visual/table.stl" />
+        </geometry>
+        <material name="">
+          <color rgba="1.0 0.0 0.0 1.0"/>
+          <texture filename=""/>
+        </material>
+      </visual>
+      <collision>
+        <origin xyz="0.0 0.0 0.0" rpy="0.0 0.0 0.0"/>
+        <geometry>
+          <mesh filename="package://ur5_description/meshes/ur5/collision/table.stl" />
+        </geometry>
+      </collision>
+  </link>
+    <link name="place_table">
       <inertial>
         <mass value="0.1" />

File: src/ur5_description/urdf/ur5_robot.urdf.xacro (robot description, xacro)
@@ -22,12 +22,17 @@
     <origin xyz="0.0 0.0 0.0" rpy="0.0 0.0 0.0" />
   </joint>
-  <joint name="world_table" type="fixed">
+  <joint name="world_pick_table" type="fixed">
     <parent link="world" />
-    <child link = "table" />
-    <origin xyz="0.7 0.0 0.0" rpy="0.0 0.0 0.0" />
+    <child link = "pick_table" />
+    <origin xyz="0.1 -0.6 0.0" rpy="0.0 0.0 0.0" />
+  </joint>
+  <joint name="world_place_table" type="fixed">
+    <parent link="world" />
+    <child link = "place_table" />
+    <origin xyz="0.01 0.6 0.0" rpy="0.0 0.0 0.0" />
   </joint>
   <xacro:include filename="$(find ur5_description)/urdf/camera.xacro"/>
   <!-- x = 0.5 the best value -->
-  <xacro:kinect_camera prefix="camera1" parent_link="world" xyz="0.7 0 2" rpy="0 0.3 0"/>
+  <xacro:kinect_camera prefix="camera1" parent_link="world" xyz="0.7 0 2" rpy="0 -0.3 0"/>
   <xacro:include filename="$(find ur5_description)/urdf/vacuum_gripper.xacro"/>
   <xacro:gripper parent_link="wrist_3_link" xyz="0 0.0823 0" rpy="0 0 ${M_PI/2}"/>
