Commit message: working with actor

File: src/ur5_description/urdf/camera.xacro (robot description, xacro)
@@ -55,10 +55,10 @@
             <always_on>true</always_on>
             <visualize>true</visualize>
-            <update_rate>10.0</update_rate>
+            <update_rate>20.0</update_rate>
             <camera name="kinetic">
             <horizontal_fov>1.047197</horizontal_fov>
             <image>
                 <!-- openni_kinect plugin works only with BGR8 -->
-                <format>L8</format>
+                <format>BGR8</format>
                 <width>640</width>
                 <height>480</height>
@@ -66,5 +66,5 @@
             <clip>
                 <near>0.1</near>
-                <far>2</far>
+                <far>5</far>
             </clip>
             </camera>
@@ -72,5 +72,5 @@
             <baseline>0.2</baseline>
             <alwaysOn>true</alwaysOn>
-            <updateRate>10.0</updateRate>
+            <updateRate>20.0</updateRate>
             <cameraName>${prefix}</cameraName>
             <imageTopicName>rgb/image_raw</imageTopicName>
@@ -80,10 +80,10 @@
             <pointCloudTopicName>depth_registered/points</pointCloudTopicName>
             <frameName>${prefix}_kinect_depth_optical_frame</frameName>
-            <pointCloudCutoff>0.1</pointCloudCutoff>
-            <pointCloudCutoffMax>2</pointCloudCutoffMax>
+            <pointCloudCutoff>0.5</pointCloudCutoff>
+            <pointCloudCutoffMax>3</pointCloudCutoffMax>
             <CxPrime>0</CxPrime>
             <Cx>0</Cx>
             <Cy>0</Cy>
-            <focalLength>0</focalLength>
+            <focalLength>1</focalLength>
             <hackBaseline>0</hackBaseline>
             </plugin>

File: src/ur5_description/urdf/ur5.urdf.xacro (robot description, xacro)
@@ -13,5 +13,5 @@
   </xacro:macro>
   <xacro:macro name="ur5_robot" params="prefix joint_limited
-    shoulder_pan_lower_limit:=${-pi}    shoulder_pan_upper_limit:=${pi}
+    shoulder_pan_lower_limit:=${-1}    shoulder_pan_upper_limit:=${pi+1}
     shoulder_lift_lower_limit:=${-pi}    shoulder_lift_upper_limit:=${pi}
     elbow_joint_lower_limit:=${-pi}    elbow_joint_upper_limit:=${pi}
@@ -168,5 +168,5 @@
       <parent link="pedestal"/>
       <child link="base_link"/>
-      <origin xyz="-0.124 0 0.95" rpy="0 0 0"/>
+      <origin xyz="-0.124 0 0.95" rpy="0 0 ${-radians(90)}"/>
     </joint>
     <link name="${prefix}base_link" >

File: src/ur5_description/urdf/ur5_robot.urdf.xacro (robot description, xacro)
@@ -8,5 +8,5 @@
   <xacro:include filename="$(find ur5_description)/urdf/ur5.urdf.xacro" />
   <!-- arm -->
-  <xacro:ur5_robot prefix="" joint_limited="false"
+  <xacro:ur5_robot prefix="" joint_limited="true"
     transmission_hw_interface="$(arg transmission_hw_interface)"
   />
@@ -34,5 +34,5 @@
   <xacro:include filename="$(find ur5_description)/urdf/camera.xacro"/>
   <!-- x = 0.5 the best value -->
-  <xacro:kinect_camera prefix="camera1" parent_link="world" xyz="0.7 0 2" rpy="0 -0.3 0"/>
+  <xacro:kinect_camera prefix="camera1" parent_link="world" xyz="0.8 2.5 0.8" rpy="0 ${-M_PI/2} ${-M_PI/2}"/>
   <xacro:include filename="$(find ur5_description)/urdf/vacuum_gripper.xacro"/>
   <xacro:gripper parent_link="wrist_3_link" xyz="0 0.0823 0" rpy="0 0 ${M_PI/2}"/>
